Commit message: First generated Noetic Ur5e Movit package!
No errors

File: ur5_ws/src/robotiq/robotiq_2f_85_gripper_visualization/urdf/robotiq_arg2f_85_macro.xacro (robot description, xacro)
@@ -180,5 +180,7 @@
     </xacro:macro>
     <!-- base link -->
-    <link name="${prefix}base_link"/>
+    <link name="${prefix}base_link">
+      <parent link="drawers_box" />
+    </link>
     <joint name="${prefix}base_link-${prefix}robotiq_arg2f_base_link" type="fixed">
       <parent link="${prefix}base_link" />

File: ur5_ws/src/universal_robot/ur_description/urdf/inc/ur_macro.xacro (robot description, xacro)
@@ -64,5 +64,7 @@
     <xacro:ur_arm_transmission prefix="${prefix}" hw_interface="${transmission_hw_interface}" />
     <!-- links: main serial chain -->
-    <link name="${prefix}base_link"/>
+    <link name="${prefix}base_link">
+          <parent link="drawers_box" />
+    </link>
     <link name="${prefix}base_link_inertia">
       <visual>

File: ur5_ws/src/ur5e2f/urdf/ur5e2f.urdf.xacro (robot description, xacro)
@@ -40,5 +40,5 @@
         <origin xyz="0.0 0.0 0.0" rpy="0.0 0.0 1.57"/>
         <parent link="tool0"/>
-        <child link="gripper-robotiq_arg2f_base_link"/>
+        <child link="gripper-base_link"/>
         <axis xyz="0.0 0.0 1.0"/>
     </joint>
