Commit message: Solved duplicated base_link problem
[ERROR] [1683900943.824225813]: Failed to find root link: Two root links found: [drawers_box] and [gripper-base_link]

File: ur5_ws/src/robotiq/robotiq_2f_85_gripper_visualization/urdf/robotiq_arg2f_85.xacro (robot description, xacro)
@@ -7,5 +7,5 @@
   <!-- gripper -->
   <xacro:robotiq_arg2f_85
-    prefix=""
+    prefix="gripper-"
     transmission_hw_interface="$(arg transmission_hw_interface)"/>
 </robot>

File: ur5_ws/src/ur5e2f/urdf/ur5e2f.urdf.xacro (robot description, xacro)
@@ -40,5 +40,5 @@
         <origin xyz="0.0 0.0 0.0" rpy="0.0 0.0 1.57"/>
         <parent link="tool0"/>
-        <child link="robotiq_arg2f_base_link"/>
+        <child link="gripper-robotiq_arg2f_base_link"/>
         <axis xyz="0.0 0.0 1.0"/>
     </joint>

Commit message: Loding model in Rviz; Issue with Gazebo simulation

File: ur5_ws/src/robotiq/robotiq_2f_85_gripper_visualization/urdf/robotiq_arg2f_85.xacro (robot description, xacro)
@@ -7,5 +7,5 @@
   <!-- gripper -->
   <xacro:robotiq_arg2f_85
-    prefix="gripper-"
+    prefix="gripper_"
     transmission_hw_interface="$(arg transmission_hw_interface)"/>
 </robot>

File: ur5_ws/src/ur5e2f/urdf/ur5e2f.urdf.xacro (robot description, xacro)
@@ -40,5 +40,5 @@
         <origin xyz="0.0 0.0 0.0" rpy="0.0 0.0 1.57"/>
         <parent link="tool0"/>
-        <child link="gripper-base_link"/>
+        <child link="gripper_base_link"/>
         <axis xyz="0.0 0.0 1.0"/>
     </joint>
