Commit message: Safe state before solution attempt

File: ur5_ws/src/ur5e2f/urdf/ur5e2f.urdf.xacro (robot description, xacro)
@@ -3,9 +3,4 @@
     <!--Create the drawers box-->
     <link name="drawers_box">
-        <inertial>
-            <origin xyz="0.0 0.0 0.505" rpy="0.0 0.0 0.0"/>
-            <mass value="50.0"/>
-            <inertia ixx="10.0" ixy="10.0" ixz="10.0" iyy="10.0" iyz="10.0" izz="10.0"/>
-        </inertial>
         <visual>
             <origin xyz="0.0 0.0 0.505" rpy="0.0 0.0 0.0"/>

Commit message: Correction to the MoveIt pack configuration

File: ur5_ws/src/ur5e2f/urdf/ur5e2f.urdf.xacro (robot description, xacro)
@@ -3,4 +3,9 @@
     <!--Create the drawers box-->
     <link name="drawers_box">
+        <inertial>
+            <origin xyz="0.0 0.0 0.505" rpy="0.0 0.0 0.0"/>
+            <mass value="50.0"/>
+            <inertia ixx="10.0" ixy="10.0" ixz="10.0" iyy="10.0" iyz="10.0" izz="10.0"/>
+        </inertial>
         <visual>
             <origin xyz="0.0 0.0 0.505" rpy="0.0 0.0 0.0"/>

Commit message: Base for version 3

File: ur5_ws/src/ur5e2f/urdf/ur5e2f.urdf.xacro (robot description, xacro)
@@ -1,4 +1,4 @@
 <?xml version="1.0"?>
-<robot xmlns:xacro="http://ros.org/wiki/xacro" name="sud_robot">
+<robot xmlns:xacro="http://ros.org/wiki/xacro" name="ur5e_robotiq">
     <!--Create the drawers box-->
     <link name="drawers_box">
@@ -31,4 +31,11 @@
         <child link="base_link"/>
         <axis xyz="0.0 0.0 1.0"/>
+    </joint>
+    <!--Couple the Drawers to the world-->
+    <link name="world"/>
+        <joint name="world_joint" type="fixed">
+        <parent link="world"/>
+        <child link="drawers_box"/>
+        <origin xyz="0 0 0" rpy="0 0 0"/>
     </joint>
     <!--Import the ur5e robot-->
