Commit message: Base MoveIt pack v.3.0

File: ur5_ws/src/ur5e_robotiq_moveit_config/config/gazebo_ur5e_robotiq.urdf (robot description, URDF)
Before this commit: robot sud_robot, 25 links, 24 joints
Links:
- added link world
Joints:
- added joint world_joint: type fixed, parent world, child drawers_box, origin xyz=0 0 0 rpy=0 0 0
