Commit message: Collision Update

File: ur5_ws/src/ur5e2f_hang/urdf/frame.xacro (robot description, xacro)
@@ -15,5 +15,5 @@
       <origin rpy="0 0 0" xyz="0 0 0"/>
       <geometry>
-        <box size="0.94 1.46 1"/>
+        <box size="0.94 1.46 0.005"/>
       </geometry>
     </collision>
@@ -122,5 +122,5 @@
       <origin rpy="0 0 0" xyz="0 0 0"/>
       <geometry>
-        <box size="0.94 1.46 1"/>
+        <box size="0.94 1.46 0.005"/>
       </geometry>
     </collision>

Commit message: Added colisions for the edges of the box

File: ur5_ws/src/ur5e2f_hang/urdf/frame.xacro (robot description, xacro)
@@ -31,7 +31,7 @@
     </visual>
     <collision>
-      <origin rpy="0 0 0" xyz="0 0 0"/>
+      <origin rpy="0 0 0" xyz="0.42 0 0"/>
       <geometry>
-        <box size="0.05 0.05 1.1"/>
+        <box size="0.94 0.05 1.1"/>
       </geometry>
     </collision>
@@ -53,7 +53,7 @@
     </visual>
     <collision>
-      <origin rpy="0 0 0" xyz="0 0 0"/>
+      <origin rpy="0 0 0" xyz="0 0.68 0"/>
       <geometry>
-        <box size="0.05 0.05 1.1"/>
+        <box size="0.05 1.46 1.1"/>
       </geometry>
     </collision>
@@ -75,7 +75,7 @@
     </visual>
     <collision>
-      <origin rpy="0 0 0" xyz="0 0 0"/>
+      <origin rpy="0 0 0" xyz="0 -0.68 0"/>
       <geometry>
-        <box size="0.05 0.05 1.1"/>
+        <box size="0.05 1.46 1.1"/>
       </geometry>
     </collision>
@@ -97,7 +97,7 @@
     </visual>
     <collision>
-      <origin rpy="0 0 0" xyz="0 0 0"/>
+      <origin rpy="0 0 0" xyz="-0.42 0 0"/>
       <geometry>
-        <box size="0.05 0.05 1.1"/>
+        <box size="0.94 0.05 1.1"/>
       </geometry>
     </collision>

File: ur5_ws/src/ur5e2f_hang/urdf/ur5e2f.urdf.xacro (robot description, xacro)
@@ -9,5 +9,5 @@
     <!--Join the UR5e with the Drawers Box-->
     <joint name="block_ur5_connection" type="fixed">
-        <origin xyz="0 0 -0.005" rpy="0 ${radians(180)} 0"/>
+        <origin xyz="0 0 -0.005" rpy="0 ${radians(180)} ${radians(90)}"/>
         <parent link="top_link"/>
         <child link="base_link"/>

Commit message: Update to rig thickness to better represent reality

File: ur5_ws/src/ur5e2f_hang/urdf/frame.xacro (robot description, xacro)
@@ -6,5 +6,5 @@
       <origin rpy="0 0 0" xyz="0 0 0"/>
       <geometry>
-        <box size="0.94 1.46 0.005"/>
+        <box size="0.94 1.46 0.04"/>
       </geometry>
       <material name="white">
@@ -15,5 +15,5 @@
       <origin rpy="0 0 0" xyz="0 0 0"/>
       <geometry>
-        <box size="0.94 1.46 0.005"/>
+        <box size="0.94 1.46 0.04"/>
       </geometry>
     </collision>
@@ -38,5 +38,5 @@
   </link>
   <joint name="joint_1" type="fixed">
-    <origin rpy="0 0 0" xyz="-0.42 -0.68 0.55"/>
+    <origin rpy="0 0 0" xyz="-0.42 -0.68 0.57"/>
     <parent link="frame_base_link"/>
     <child link="leg_1"/>
@@ -60,5 +60,5 @@
   </link>
   <joint name="joint_2" type="fixed">
-    <origin rpy="0 0 0" xyz="0.42 -0.68 0.55"/>
+    <origin rpy="0 0 0" xyz="0.42 -0.68 0.57"/>
     <parent link="frame_base_link"/>
     <child link="leg_2"/>
@@ -82,5 +82,5 @@
   </link>
   <joint name="joint_3" type="fixed">
-    <origin rpy="0 0 0" xyz="-0.42 0.68 0.55"/>
+    <origin rpy="0 0 0" xyz="-0.42 0.68 0.57"/>
     <parent link="frame_base_link"/>
     <child link="leg_3"/>
@@ -104,5 +104,5 @@
   </link>
   <joint name="joint_4" type="fixed">
-    <origin rpy="0 0 0" xyz="0.42 0.68 0.55"/>
+    <origin rpy="0 0 0" xyz="0.42 0.68 0.57"/>
     <parent link="frame_base_link"/>
     <child link="leg_4"/>
@@ -113,5 +113,5 @@
       <origin rpy="0 0 0" xyz="0 0 0"/>
       <geometry>
-        <box size="0.94 1.46 0.005"/>
+        <box size="0.94 1.46 0.055"/>
       </geometry>
       <material name="white">
@@ -122,10 +122,10 @@
       <origin rpy="0 0 0" xyz="0 0 0"/>
       <geometry>
-        <box size="0.94 1.46 0.005"/>
+        <box size="0.94 1.46 0.055"/>
       </geometry>
     </collision>
   </link>
   <joint name="joint_top" type="fixed">
-    <origin rpy="0 0 0" xyz="0.42 -0.68 0.55"/>
+    <origin rpy="0 0 0" xyz="0.42 -0.68 0.57"/>
     <parent link="leg_3"/>
     <child link="top_link"/>

File: ur5_ws/src/ur5e2f_hang/urdf/ur5e2f.urdf.xacro (robot description, xacro)
@@ -9,5 +9,5 @@
     <!--Join the UR5e with the frame Box-->
     <joint name="block_ur5_connection" type="fixed">
-        <origin xyz="0 0 -0.005" rpy="0 ${radians(180)} ${radians(90)}"/>
+        <origin xyz="0 0 -0.0275" rpy="0 ${radians(180)} ${radians(90)}"/>
         <parent link="top_link"/>
         <child link="base_link"/>

File: ur5_ws/src/ur5e_robotiq_hang_moveit_config_V2/config/gazebo_ur5e_robotiq.urdf (robot description, URDF)
Before this commit: robot ur5e_robotiq, 30 links, 29 joints
Links:
- link frame_base_link: geometry collision box size=0.94 1.46 0.04; visual box size=0.94 1.46 0.04
- link leg_1: geometry collision box size=0.94 0.05 1.115; visual box size=0.05 0.05 1.115
- link leg_2: geometry collision box size=0.05 1.46 1.115; visual box size=0.05 0.05 1.115
- link leg_3: geometry collision box size=0.05 1.46 1.115; visual box size=0.05 0.05 1.115
- link leg_4: geometry collision box size=0.94 0.05 1.115; visual box size=0.05 0.05 1.115
- link top_link: geometry collision box size=0.94 1.46 0.04; visual box size=0.94 1.46 0.04
Joints:
- joint block_ur5_connection: origin xyz=0 0 -0.005 rpy=0 3.141592653589793 1.5707963267948966 -> xyz=0 0 -0.04 rpy=0 3.141592653589793 1.5707963267948966
- joint joint_1: origin xyz=-0.42 -0.68 0.55 rpy=0 0 0 -> xyz=-0.42 -0.68 0.5575 rpy=0 0 0
- joint joint_2: origin xyz=0.42 -0.68 0.55 rpy=0 0 0 -> xyz=0.42 -0.68 0.5575 rpy=0 0 0
- joint joint_3: origin xyz=-0.42 0.68 0.55 rpy=0 0 0 -> xyz=-0.42 0.68 0.5575 rpy=0 0 0
- joint joint_4: origin xyz=0.42 0.68 0.55 rpy=0 0 0 -> xyz=0.42 0.68 0.5575 rpy=0 0 0
- joint joint_top: origin xyz=0.42 -0.68 0.55 rpy=0 0 0 -> xyz=0.42 -0.68 0.5575 rpy=0 0 0
