Commit message: Pre implementation of carthesian paths

File: ur5_ws/src/ur5e_robotiq_hang_moveit_config_V2/config/gazebo_ur5e_robotiq.urdf (robot description, URDF)
Before this commit: robot ur5e_robotiq, 30 links, 29 joints
Links:
- removed link gripper_tip
- link leg_1: geometry collision box size=0.94 0.05 1.1; visual box size=0.05 0.05 1.1
- link leg_2: geometry collision box size=0.05 1.46 1.1; visual box size=0.05 0.05 1.1
- link leg_3: geometry collision box size=0.05 1.46 1.1; visual box size=0.05 0.05 1.1
- link leg_4: geometry collision box size=0.94 0.05 1.1; visual box size=0.05 0.05 1.1
- link top_link: geometry collision box size=0.94 1.46 0.055; visual box size=0.94 1.46 0.055
Joints:
- removed joint joint_gripper_tip
- joint block_ur5_connection: origin xyz=0 0 -0.04 rpy=0 3.141592653589793 1.5707963267948966 -> xyz=0 0 -0.0275 rpy=0 3.141592653589793 1.5707963267948966
- joint joint_1: origin xyz=-0.42 -0.68 0.5575 rpy=0 0 0 -> xyz=-0.42 -0.68 0.57 rpy=0 0 0
- joint joint_2: origin xyz=0.42 -0.68 0.5575 rpy=0 0 0 -> xyz=0.42 -0.68 0.57 rpy=0 0 0
- joint joint_3: origin xyz=-0.42 0.68 0.5575 rpy=0 0 0 -> xyz=-0.42 0.68 0.57 rpy=0 0 0
- joint joint_4: origin xyz=0.42 0.68 0.5575 rpy=0 0 0 -> xyz=0.42 0.68 0.57 rpy=0 0 0
- joint joint_top: origin xyz=0.42 -0.68 0.5575 rpy=0 0 0 -> xyz=0.42 -0.68 0.57 rpy=0 0 0
